Commit message: integrate Ackermann steering, added ros bridge,fixed bugs with the physics

File: cmh_description/urdf/car.urdf.xacro (robot description, xacro)
@@ -33,4 +33,30 @@
     <!-- Wheels -->
     <xacro:wheels chassis_width="1.6" wheelbase="1.580"/>
+    <!-- Gazebo Harmonic Ackermann Drive Plugin -->
+    <gazebo>
+        <plugin filename="gz-sim-ackermann-steering-system" name="gz::sim::systems::AckermannSteering">
+            <left_joint>rear_left_wheel_joint</left_joint>
+            <right_joint>rear_right_wheel_joint</right_joint>
+            <left_steering_joint>left_steering_hinge_joint</left_steering_joint>
+            <right_steering_joint>right_steering_hinge_joint</right_steering_joint>
+            <wheel_separation>1.6</wheel_separation>
+            <wheel_base>1.580</wheel_base>
+            <wheel_radius>0.2525</wheel_radius>
+            <steering_limit>0.5</steering_limit> <!-- Radians (~28 degrees) -->
+            <topic>/cmd_vel</topic>
+            <!-- Odometry Publishing -->
+            <kingpin_width>1.3</kingpin_width>
+            <odom_topic>/odom</odom_topic>
+            <max_velocity>200.0</max_velocity>
+            <max_acceleration>2.0</max_acceleration>
+            <min_acceleration>-5.0</min_acceleration>
+            <odom_publish_frequency>50</odom_publish_frequency>
+            <frame_id>odom</frame_id>
+            <child_frame_id>base_footprint</child_frame_id>
+        </plugin>
+        <plugin filename="gz-sim-joint-state-publisher-system" name="gz::sim::systems::JointStatePublisher">
+            <topic>/joint_states</topic>
+        </plugin>
+    </gazebo>
     <!-- *********************************************** -->
     <!--                 MAIN SENSORS                    -->

File: cmh_description/urdf/wheels.urdf.xacro (robot description, xacro)
@@ -12,5 +12,6 @@
     <xacro:property name="wheel_friction_mu1" value="2"/>
     <xacro:property name="wheel_friction_mu2" value="2"/>
-    <xacro:property name="wheel_friction_kp" value="1e8"/>
+    <xacro:property name="wheel_friction_kp" value="100000000.0"/>
+    <xacro:property name="wheel_friction_kd" value="100.0"/>
     <xacro:property name="steering_hinge_mass" value="1"/>
     <!-- ***************** -->
@@ -45,9 +46,24 @@
       </link>
       <gazebo reference="${lr_prefix}_${fr_prefix}_wheel">
-        <material>Gazebo/Black</material>
-        <mu1>${wheel_friction_mu1}</mu1>
-        <mu2>${wheel_friction_mu2}</mu2>
-        <!-- <minDepth>0.005</minDepth> -->
-        <kp>${wheel_friction_kp}</kp>
+        <material name="black">
+          <color rgba="0.1 0.1 0.1 1"/>
+        </material>
+        <collision>
+          <surface>
+            <friction>
+              <ode>
+                <mu>${wheel_friction_mu1}</mu>
+                <mu2>${wheel_friction_mu2}</mu2>
+                <fdir1>1 0 0</fdir1>
+              </ode>
+            </friction>
+            <contact>
+              <ode>
+                <kp>${wheel_friction_kp}</kp>
+                <kd>${wheel_friction_kd}</kd>
+              </ode>
+            </contact>
+          </surface>
+        </collision>
       </gazebo>
     </xacro:macro>
@@ -87,5 +103,5 @@
         <child link="${lr_prefix}_front_wheel"/>
         <axis xyz="0 1 0"/>
-        <limit lower="0" upper="0" effort="10000000" velocity="1000000"/>
+        <limit effort="10000000" velocity="1000000"/>
       </joint>
       <xacro:wheel lr_prefix="${lr_prefix}" fr_prefix="front"/>
@@ -102,5 +118,5 @@
         <child link="${lr_prefix}_rear_wheel"/>
         <axis xyz="0 1 0"/>
-        <limit lower="0" upper="0" effort="10000000" velocity="1000000"/>
+        <limit  effort="10000000" velocity="1000000"/>
       </joint>
       <xacro:wheel lr_prefix="${lr_prefix}" fr_prefix="rear"/>

Commit message: refactor: reorganize sensor architecture, update vehicle mass, and expand simulation track model

File: cmh_description/urdf/car.urdf.xacro (robot description, xacro)
@@ -1,4 +1,4 @@
 <?xml version="1.0"?>
-<robot name="eufs" xmlns:xacro="http://www.ros.org/wiki/xacro">
+<robot name="cmh" xmlns:xacro="http://www.ros.org/wiki/xacro">
     <!-- ***************** -->
     <!-- Config parameters -->
@@ -11,8 +11,6 @@
     <!-- ***************** -->
     <xacro:property name="PI" value="3.1415926535897931"/>
-    <!-- If the gazebo_ros_race_car_model should publish the ground truth tf -->
-    <xacro:arg name="publish_tf" default="false"/>
     <!-- If the perception stack should be simulated or if sensors should be used -->
-    <xacro:arg name="simulate_perception" default="true"/>
+    <xacro:arg name="simulate_perception" default="false"/>
     <!-- ***************** -->
     <!-- Imported elements -->
@@ -20,8 +18,8 @@
     <!--  Import the wheels  -->
     <xacro:include filename="$(find cmh_description)/urdf/wheels.urdf.xacro"/>
-    <!-- Import EUFS base element with the chassis -->
+    <!-- Import CMH base element with the chassis -->
     <xacro:include filename="$(find cmh_description)/urdf/cmh_base.urdf.xacro" />
-    <!-- Import all available sensors
-    <xacro:include filename="$(find eufs_sensors)/urdf/all_sensors.urdf.xacro" /> -->
+    <!-- Import all available sensors -->
+    <xacro:include filename="$(find cmh_sensors)/urdf/all_sensors.urdf.xacro" />
     <!--  Include the plugins
     <xacro:include filename="$(find eufs_plugins)/urdf/eufs_plugins.gazebo.xacro" /> -->
@@ -63,26 +61,8 @@
     <!-- *********************************************** -->
     <!--     LOCATIONS: (XYZ)
-    IMU: 0.0 0.0 0.170
-    GPS: -0.110 0.0 0.9
-    LIDAR: 1.700 0.0 -0.150
-    STEREO CAM: -0.110 0.0 0.800
-    <xacro:sensor_imu parent="chassis" prefix="sbg_imu" topic_prefix="">
-        <origin xyz="0.0 0.0 0.0" rpy="0 0 0"/>
-    </xacro:sensor_imu>
-    <xacro:sensor_gps parent="chassis" prefix="gps">
-        <origin xyz="0.0 0.0 0.4" rpy="0 0 0"/>
-    </xacro:sensor_gps>
-    <xacro:VLP-16R parent="chassis" name="velodyne" topic="/velodyne_points" hz="10" active="$(arg simulate_perception)">
-        <origin xyz="-0.15 0.0 0.79" rpy="0 ${1*M_PI/180.0} 0"/>
-    </xacro:VLP-16R>
-    <xacro:zed_camera parent="chassis" prefix="zed" active="$(arg simulate_perception)">
-        <origin xyz="-0.08 0.0 0.76" rpy="0 0 0"/>
-    </xacro:zed_camera>
-    <xacro:sensor_imu parent="chassis" prefix="zed_imu" topic_prefix="/camera">
-        <origin xyz="-0.08 0.0 0.76" rpy="0 0 0"/>
-    </xacro:sensor_imu>
-    <xacro:sensor_magnetometer parent="chassis" prefix="sbg">
-        <origin xyz="0.0 0.0 0.0" rpy="0 0 0"/>
-    </xacro:sensor_magnetometer>
+    CAM: -0.110 0.0 0.800
     -->
+    <xacro:monocular_camera parent="chassis" prefix="camera" active="$(arg simulate_perception)">
+        <origin xyz="-0.08 0.0 0.76" rpy="0 0.1 0"/>
+    </xacro:monocular_camera>
 </robot>

File: cmh_description/urdf/cmh_base.urdf.xacro (robot description, xacro)
@@ -33,5 +33,5 @@
         <origin xyz="0 0 0" rpy="0 0 0" />
         <geometry>
-          <mesh filename="${chassis_mesh}"/>
+          <box size="1.0 0.6 0.3"/>
         </geometry>
       </collision>
