Commit message: migrated to ros2 lyrical distribution, improved track rendering and real-time factor by making cones static and rendering a minimal_car instead

File: cmh_description/urdf/car.urdf.xacro (robot description, xacro)
@@ -30,6 +30,6 @@
     <xacro:cmh_base chassis_mesh="file://$(find cmh_description)/meshes/sisu-20d.dae"/>
     <!-- Wheels -->
-    <xacro:wheels chassis_width="1.6" wheelbase="1.580"/>
-    <!-- Gazebo Harmonic Ackermann Drive Plugin -->
+    <xacro:wheels track_width="${config['kinematics']['axle_width']}" wheelbase="${config['kinematics']['l']}"/>
+    <!-- Gazebo Ackermann Drive Plugin (geometry and limits come from the config file) -->
     <gazebo>
         <plugin filename="gz-sim-ackermann-steering-system" name="gz::sim::systems::AckermannSteering">
@@ -38,15 +38,16 @@
             <left_steering_joint>left_steering_hinge_joint</left_steering_joint>
             <right_steering_joint>right_steering_hinge_joint</right_steering_joint>
-            <wheel_separation>1.6</wheel_separation>
-            <wheel_base>1.580</wheel_base>
-            <wheel_radius>0.2525</wheel_radius>
-            <steering_limit>0.5</steering_limit> <!-- Radians (~28 degrees) -->
+            <wheel_separation>${config['kinematics']['axle_width']}</wheel_separation>
+            <kingpin_width>${config['kinematics']['axle_width']}</kingpin_width>
+            <wheel_base>${config['kinematics']['l']}</wheel_base>
+            <wheel_radius>${config['tire']['radius']}</wheel_radius>
+            <steering_limit>${config['input_ranges']['steering']['max']}</steering_limit> <!-- Radians -->
             <topic>/cmd_vel</topic>
+            <max_velocity>${config['input_ranges']['velocity']['max']}</max_velocity>
+            <max_acceleration>${config['input_ranges']['acceleration']['max']}</max_acceleration>
+            <min_acceleration>${config['input_ranges']['acceleration']['min']}</min_acceleration>
             <!-- Odometry Publishing -->
-            <kingpin_width>1.3</kingpin_width>
             <odom_topic>/odom</odom_topic>
-            <max_velocity>200.0</max_velocity>
-            <max_acceleration>2.0</max_acceleration>
-            <min_acceleration>-5.0</min_acceleration>
+            <tf_topic>/tf</tf_topic>
             <odom_publish_frequency>50</odom_publish_frequency>
             <frame_id>odom</frame_id>
@@ -63,5 +64,5 @@
     CAM: -0.110 0.0 0.800
     -->
-    <xacro:monocular_camera parent="chassis" prefix="camera" active="$(arg simulate_perception)">
+    <xacro:monocular_camera parent="chassis" prefix="camera" simulate_perception="$(arg simulate_perception)">
         <origin xyz="-0.08 0.0 0.76" rpy="0 0.1 0"/>
     </xacro:monocular_camera>

File: cmh_description/urdf/cmh_base.urdf.xacro (robot description, xacro)
@@ -2,5 +2,5 @@
 <robot name="cmh" xmlns:xacro="http://www.ros.org/wiki/xacro">
   <xacro:macro name="cmh_base" params="chassis_mesh">
-    <xacro:property name="wheel_diameter" value="0.505"/>
+    <xacro:property name="wheel_diameter" value="${2 * config['tire']['radius']}"/>
     <!-- BASE FOOTPRINT -->
     <link name="base_footprint"/>
@@ -30,4 +30,5 @@
             izz="47.9" />
       </inertial>
+      <!--
       <collision>
         <origin xyz="0 0 0" rpy="0 0 0" />
@@ -36,4 +37,5 @@
         </geometry>
       </collision>
+      -->
     </link>
   </xacro:macro>

File: cmh_description/urdf/wheels.urdf.xacro (robot description, xacro)
@@ -2,5 +2,5 @@
 <robot name="wheels" xmlns:xacro="http://www.ros.org/wiki/xacro">
   <xacro:macro name="wheels"
-               params="chassis_width wheelbase">
+               params="track_width wheelbase">
     <!-- ********** -->
     <!-- Parameters -->
@@ -8,5 +8,5 @@
     <xacro:property name="degrees_90" value="1.5708"/>
     <xacro:property name="wheel_mass" value="10.0"/>
-    <xacro:property name="wheel_diameter" value="0.505"/>
+    <xacro:property name="wheel_diameter" value="${2 * config['tire']['radius']}"/>
     <xacro:property name="wheel_width" value="0.2"/>
     <xacro:property name="wheel_friction_mu1" value="2"/>
@@ -25,8 +25,8 @@
           <mass value="${wheel_mass}"/>
           <inertia
-              ixx="0.3"
+              ixx="0.2"
               ixy="0"
               ixz="0"
-              iyy="0.2"
+              iyy="0.3"
               iyz="0"
               izz="0.2"   />
@@ -46,7 +46,4 @@
       </link>
       <gazebo reference="${lr_prefix}_${fr_prefix}_wheel">
-        <material name="black">
-          <color rgba="0.1 0.1 0.1 1"/>
-        </material>
         <collision>
           <surface>
@@ -76,5 +73,5 @@
       <joint name="${lr_prefix}_steering_hinge_joint" type="revolute">
         <origin xyz="${wheelbase / 2}
-                     ${lr_reflect * ((chassis_width - wheel_width) / 2)}
+                     ${lr_reflect * track_width / 2}
                      0"
                 rpy="0 0 0"/>
@@ -112,5 +109,5 @@
       <joint name="rear_${lr_prefix}_wheel_joint" type="continuous">
         <origin xyz="${-1 * wheelbase / 2}
-                     ${lr_reflect * ((chassis_width - wheel_width) / 2)}
+                     ${lr_reflect * track_width / 2}
                      0"
                 rpy="0 0 0"/>

File: cmh_sensors/urdf/monocular_camera.urdf.xacro (robot description, xacro)
@@ -1,5 +1,5 @@
 <?xml version="1.0"?>
 <robot name="monocular_camera" xmlns:xacro="http://www.ros.org/wiki/xacro">
-  <xacro:macro name="monocular_camera" params="prefix parent *origin active">
+  <xacro:macro name="monocular_camera" params="prefix parent *origin simulate_perception">
     <joint name="${prefix}_base_joint" type="fixed">
       <xacro:insert_block name="origin"/>
@@ -18,5 +18,6 @@
       </visual>
     </link>
-    <xacro:unless value="${active}">
+    <!-- The camera sensor only exists when perception is simulated -->
+    <xacro:if value="${simulate_perception}">
       <gazebo reference="${prefix}_center">
         <sensor type="camera" name="${prefix}_monocular_rgb_camera">
@@ -25,6 +26,6 @@
           <visualize>true</visualize>
           <topic>${prefix}/image_raw</topic>
+          <gz_frame_id>${prefix}_center</gz_frame_id>
           <camera name="${prefix}_front">
-            <horizontal_fov>1.39</horizontal_fov>
             <image>
               <width>640</width>
@@ -32,4 +33,13 @@
               <format>R8G8B8</format>
             </image>
+            <lens>
+              <intrinsics>
+                <fx>500.0</fx>
+                <fy>500.0</fy>
+                <cx>320.0</cx>
+                <cy>240.0</cy>
+                <s>0.0</s>
+              </intrinsics>
+            </lens>
             <clip>
               <near>0.05</near>
@@ -44,5 +54,5 @@
         </sensor>
       </gazebo>
-    </xacro:unless>
+    </xacro:if>
   </xacro:macro>
 </robot>
